Commit message: Setup robot with onshape-to-robot Setup behavior trees add paths

File: daybreak_robot/description/robot.urdf.xacro (robot description, xacro)
@@ -1,9 +1,18 @@
 <?xml version="1.0"?>
-<robot xmlns:xacro="http://www.ros.org/wiki/xacro" name="robot">
+<robot xmlns:xacro="http://www.ros.org/wiki/xacro" name="daybreak">
     <xacro:arg name="sim" default="false" />
     <xacro:property name="sim" value="$(arg sim)" />
+    <link name="base_link">
+    </link>
+    <joint name="chassis_link" type="fixed">
+        <parent link="base_link" />
+        <child link="chassis" />
+    </joint>
     <xacro:include filename="$(find daybreak_robot)/description/inertial_macros.xacro" />
     <xacro:include filename="$(find daybreak_robot)/description/colors.xacro" />
-    <xacro:include filename="$(find daybreak_robot)/description/robot_drivetrain.xacro" />
+    <xacro:include filename="$(find daybreak_robot)/description/robot_collision.xacro" />
+    <xacro:include filename="$(find daybreak_robot)/description/robot.urdf" />
+    <xacro:include filename="$(find daybreak_robot)/description/ros2_control_drivetrain.xacro" />
+    <xacro:include filename="$(find daybreak_robot)/description/ros2_control_hammer.xacro" />
     <xacro:include filename="$(find daybreak_robot)/description/robot_core.xacro" />
     <gazebo>

File: daybreak_robot/description/ros2_control_drivetrain.xacro (robot description, xacro)
@@ -12,5 +12,5 @@
                 </xacro:unless>
             </hardware>
-            <joint name="${prefix}_wheel_rotate_joint">
+            <joint name="chassis_to_wheel_rotate_${prefix}">
                 <command_interface name="position" />
                 <state_interface name="position" />
@@ -19,5 +19,6 @@
             <transmission name="transmission1">
                 <plugin>transmission_interface/SimpleTransmission</plugin>
-                <joint name="${prefix}_wheel_rotate_joint" role="${prefix}_wheel_rotate_joint">
+                <joint name="chassis_to_wheel_rotate_${prefix}"
+                    role="chassis_to_wheel_rotate_${prefix}">
                     <mechanical_reduction>${150/7}</mechanical_reduction>
                 </joint>
@@ -34,5 +35,5 @@
                 </xacro:unless>
             </hardware>
-            <joint name="${prefix}_wheel_joint">
+            <joint name="wheel_rotate_${prefix}_to_wheel_spin_${prefix}">
                 <command_interface name="velocity" />
                 <state_interface name="position" />
@@ -41,17 +42,18 @@
             <transmission name="transmission1">
                 <plugin>transmission_interface/SimpleTransmission</plugin>
-                <joint name="${prefix}_wheel_joint" role="${prefix}_wheel_joint">
+                <joint name="wheel_rotate_${prefix}_to_wheel_spin_${prefix}"
+                    role="wheel_rotate_${prefix}_to_wheel_spin_${prefix}">
                     <mechanical_reduction>6.12</mechanical_reduction>
                 </joint>
             </transmission>
         </ros2_control>
-        <gazebo reference="${prefix}_wheel">
+        <gazebo reference="wheel_spin_${prefix}">
             <mu1>1.16</mu1>
             <mu2>1.16</mu2>
         </gazebo>
     </xacro:macro>
-    <xacro:swerve_wheel_control prefix="front_left" />
-    <xacro:swerve_wheel_control prefix="front_right" />
-    <xacro:swerve_wheel_control prefix="rear_left" />
-    <xacro:swerve_wheel_control prefix="rear_right" />
+    <xacro:swerve_wheel_control prefix="fl" />
+    <xacro:swerve_wheel_control prefix="fr" />
+    <xacro:swerve_wheel_control prefix="bl" />
+    <xacro:swerve_wheel_control prefix="br" />
 </robot>
